File: Kicad/PC-8001mk2_SD.kicad_pcb (KiCad board)
At the start: 2 copper layers, 99.9 x 95 mm, 14 parts, among them J1 Conn_02x36_Row_Letter_First, J2 Micro_SD_Card_Kit, U1 74LS04, U2 74LS30, U3 8255, U4 Arduino_Pro_Mini_5V

Commit message: Add files via upload
Parts:
- added J3: MicroSD Card Adapter, Connector_PinSocket_2.54mm:PinSocket_1x06_P2.54mm_Vertical, F.Cu at (161.3, 113.8)
- moved C4 4.05 mm to (105.7, 99.6)
- moved U3 4.05 mm to (158.4, 90.6)
- moved C2 2.00 mm to (129.0, 79.3)
- moved C3 2.00 mm to (153.8, 79.3)
- moved U1 2.00 mm to (125.2, 76.7)
- moved U2 2.00 mm to (150.0, 76.7)
Connections:
- net Net-(J2-Pad5) renamed /SCK
- net Net-(J2-Pad6) renamed /MISO
- net Net-(J2-Pad7) renamed /MOSI
- net Net-(J2-Pad8) renamed /CS
Routing:
- net GND: track 289.2 -> 249.0 mm, vias 1 -> 0
- net /D6: track 49.2 -> 74.1 mm, vias 2 -> 0
- net +5V: track 258.3 -> 234.3 mm, vias 1 -> 0
- net /MOSI: track 45.6 -> 61.0 mm
- net Net-(U3-Pad3): track 79.8 -> 93.0 mm, vias 1 -> 0
- net /~RESET: track 116.1 -> 103.0 mm
- net /~RD: track 51.6 -> 38.8 mm, vias 2 -> 1
- net /~WR: track 62.4 -> 49.9 mm, vias 3 -> 1
- net /SCK: track 51.4 -> 63.7 mm
- net /MISO: track 47.8 -> 60.1 mm
- net /~IOREQ: track 36.4 -> 24.3 mm
- net Net-(U3-Pad2): track 98.3 -> 86.3 mm
- net Net-(U3-Pad19): track 47.6 -> 59.0 mm, vias 1 -> 0
- net /CS: track 43.1 -> 53.7 mm
- net Net-(U3-Pad1): track 99.0 -> 89.9 mm
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Other:
- board text added: "PC-8001mk2_SD Rev1.1"
- board text removed: "PC-8001mk2_SD Rev1.0"
